Commit message: added b1 simulation based on bullet_utils

File: B1Env/robots/b1_raw.urdf (robot description, URDF)
Before this commit: robot b1_description, 17 links, 16 joints
Joints:
- joint FL_thigh_joint: type continuous -> revolute
- joint FR_thigh_joint: type continuous -> revolute
- joint HL_thigh_joint: type continuous -> revolute
- joint HR_thigh_joint: type continuous -> revolute

Commit message: updated b1_raw.urdf

File: B1Env/robots/b1_raw.urdf (robot description, URDF)
Before this commit: robot b1_description, 17 links, 16 joints
Links:
- added link FL_calf_rotor, mass 0.266; collision cylinder length=0.02 radius=0.05; visual cylinder length=0.02 radius=0.05
- added link FL_hip_rotor, mass 0.199; collision cylinder length=0.02 radius=0.05; visual cylinder length=0.02 radius=0.05
- added link FL_thigh_rotor, mass 0.266; collision cylinder length=0.02 radius=0.05; visual cylinder length=0.02 radius=0.05
- added link FR_calf_rotor, mass 0.266; collision cylinder length=0.02 radius=0.05; visual cylinder length=0.02 radius=0.05
- added link FR_hip_rotor, mass 0.199; collision cylinder length=0.02 radius=0.05; visual cylinder length=0.02 radius=0.05
- added link FR_thigh_rotor, mass 0.266; collision cylinder length=0.02 radius=0.05; visual cylinder length=0.02 radius=0.05
- added link HL_calf_rotor, mass 0.266; collision cylinder length=0.02 radius=0.05; visual cylinder length=0.02 radius=0.05
- added link HL_hip_rotor, mass 0.199; collision cylinder length=0.02 radius=0.05; visual cylinder length=0.02 radius=0.05
- added link HL_thigh_rotor, mass 0.266; collision cylinder length=0.02 radius=0.05; visual cylinder length=0.02 radius=0.05
- added link HR_calf_rotor, mass 0.266; collision cylinder length=0.02 radius=0.05; visual cylinder length=0.02 radius=0.05
- added link HR_hip_rotor, mass 0.199; collision cylinder length=0.02 radius=0.05; visual cylinder length=0.02 radius=0.05
- added link HR_thigh_rotor, mass 0.266; collision cylinder length=0.02 radius=0.05; visual cylinder length=0.02 radius=0.05
- link FL_calf: mass 0.207 -> 0.857; geometry collision box size=0.35 0.04 0.05; visual mesh filename=package://robots/meshes/calf.dae scale=1 1 1
- link FL_foot: mass 0.06 -> 0.05
- link FL_hip: mass 1.993 -> 2.1
- link FL_thigh: mass 0.639 -> 3.934
- link FR_calf: mass 0.207 -> 0.857; geometry collision box size=0.35 0.04 0.05; visual mesh filename=package://robots/meshes/calf.dae scale=1 1 1
- link FR_foot: mass 0.06 -> 0.05
- link FR_hip: mass 1.993 -> 2.1
- link FR_thigh: mass 0.639 -> 3.934
- link HL_calf: mass 0.207 -> 0.857; geometry collision box size=0.35 0.04 0.05; visual mesh filename=package://robots/meshes/calf.dae scale=1 1 1
- link HL_foot: mass 0.06 -> 0.05
- link HL_hip: mass 1.993 -> 2.1
- link HL_thigh: mass 0.639 -> 3.934
- link HR_calf: mass 0.207 -> 0.857; geometry collision box size=0.35 0.04 0.05; visual mesh filename=package://robots/meshes/calf.dae scale=1 1 1
- link HR_foot: mass 0.06 -> 0.05
- link HR_hip: mass 1.993 -> 2.1
- link HR_thigh: mass 0.639 -> 3.934
- link trunk: mass 9.041 -> 25
Joints:
- added joint FL_calf_rotor_joint: type fixed, parent FL_thigh, child FL_calf_rotor, origin xyz=0.0 -0.0519 0 rpy=0 0 0
- added joint FL_hip_rotor_joint: type fixed, parent trunk, child FL_hip_rotor, origin xyz=0.1955 0.072 0 rpy=0 0 0
- added joint FL_thigh_rotor_joint: type fixed, parent FL_hip, child FL_thigh_rotor, origin xyz=0.0 0.00935 0 rpy=0 0 0
- added joint FR_calf_rotor_joint: type fixed, parent FR_thigh, child FR_calf_rotor, origin xyz=0.0 0.0519 0 rpy=0 0 0
- added joint FR_hip_rotor_joint: type fixed, parent trunk, child FR_hip_rotor, origin xyz=0.1955 -0.072 0 rpy=0 0 0
- added joint FR_thigh_rotor_joint: type fixed, parent FR_hip, child FR_thigh_rotor, origin xyz=0.0 -0.00935 0 rpy=0 0 0
- added joint HL_calf_rotor_joint: type fixed, parent HL_thigh, child HL_calf_rotor, origin xyz=0.0 -0.0519 0 rpy=0 0 0
- added joint HL_hip_rotor_joint: type fixed, parent trunk, child HL_hip_rotor, origin xyz=-0.1955 0.072 0 rpy=0 0 0
- added joint HL_thigh_rotor_joint: type fixed, parent HL_hip, child HL_thigh_rotor, origin xyz=0.0 0.00935 0 rpy=0 0 0
- added joint HR_calf_rotor_joint: type fixed, parent HR_thigh, child HR_calf_rotor, origin xyz=0.0 0.0519 0 rpy=0 0 0
- added joint HR_hip_rotor_joint: type fixed, parent trunk, child HR_hip_rotor, origin xyz=-0.1955 -0.072 0 rpy=0 0 0
- added joint HR_thigh_rotor_joint: type fixed, parent HR_hip, child HR_thigh_rotor, origin xyz=0.0 -0.00935 0 rpy=0 0 0
- joint FL_hip_joint: limit lower=-0.75 upper=0.75 effort=100 velocity=20 -> lower=-0.75 upper=0.75 effort=91.0035 velocity=19.69
- joint FL_knee_joint: limit lower=-2.6 upper=-0.6 effort=100 velocity=20 -> lower=-2.6 upper=-0.6 effort=140 velocity=15.55
- joint FL_thigh_joint: limit lower=-1.0 upper=3.5 effort=100 velocity=20 -> lower=-1.0 upper=3.5 effort=93.33 velocity=23.32
- joint FR_hip_joint: limit lower=-0.75 upper=0.75 effort=100 velocity=20 -> lower=-0.75 upper=0.75 effort=91.0035 velocity=19.69
- joint FR_knee_joint: limit lower=-2.6 upper=-0.6 effort=100 velocity=20 -> lower=-2.6 upper=-0.6 effort=140 velocity=15.55
- joint FR_thigh_joint: limit lower=-1.0 upper=3.5 effort=100 velocity=20 -> lower=-1.0 upper=3.5 effort=93.33 velocity=23.32
- joint HL_hip_joint: limit lower=-0.75 upper=0.75 effort=100 velocity=20 -> lower=-0.75 upper=0.75 effort=91.0035 velocity=19.69
- joint HL_knee_joint: limit lower=-2.6 upper=-0.6 effort=100 velocity=20 -> lower=-2.6 upper=-0.6 effort=140 velocity=15.55
- joint HL_thigh_joint: limit lower=-1.0 upper=3.5 effort=100 velocity=20 -> lower=-1.0 upper=3.5 effort=93.33 velocity=23.32
- joint HR_hip_joint: limit lower=-0.75 upper=0.75 effort=100 velocity=20 -> lower=-0.75 upper=0.75 effort=91.0035 velocity=19.69
- joint HR_knee_joint: limit lower=-2.6 upper=-0.6 effort=100 velocity=20 -> lower=-2.6 upper=-0.6 effort=140 velocity=15.55
- joint HR_thigh_joint: limit lower=-1.0 upper=3.5 effort=100 velocity=20 -> lower=-1.0 upper=3.5 effort=93.33 velocity=23.32
